File: Vex_Debug.kicad_sch (KiCad schematic)
At the start: 30 parts, among them J1 USB_C_Receptacle_USB2.0, U1 ESP32-C3-MINI-1-N4, U2 NCP1117-3.3_SOT223, U3 ADM3493ARZ

Commit message: Revision 2.1 release
Parts:
- removed JP1, JP2: SolderJumper_2_Open, Jumper:SolderJumper-2_P1.3mm_Open_RoundedPad1.0x1.5mm, symbol Jumper:SolderJumper_2_Open
- removed U1: ESP32-C3-MINI-1-N4, ESP32-C3-MINI:XCVR_ESP32-C3-MINI-1-N4, symbol ESP32-C3-MINI-1-N4:ESP32-C3-MINI-1-N4
- added C7, C8: 1uF, Capacitor_SMD:C_0805_2012Metric_Pad1.18x1.45mm_HandSolder, symbol Device:C
- added R9: 5.11K, Resistor_SMD:R_0805_2012Metric_Pad1.20x1.40mm_HandSolder, symbol Device:R_US
- added SW1: RESET, Button_Switch_THT:SW_PUSH_6mm, symbol Switch:SW_Push
- added SW2: BOOT, Button_Switch_THT:SW_PUSH_6mm, symbol Switch:SW_Push
- added U1: ESP32-C3-WROOM-02-N4, ESP32-C3-WROOM:ESP32-C3-WROOM-02-N4, symbol ESP32-C3-WROOM:ESP32-C3-WROOM-02-N4
- added U4: FT234XD-R, USB-UART Bridge:FT234XD-R, symbol FTDI:FT234XD-R
Connections:
- net +3.3V: now also R7.2, R8.2, C7.1, R9.2, U1.1 (3V3), U4.4 (VCC), U4.9 (VCCIO); no longer R7.1, R8.1
- net GND: now also C7.2, C8.2, SW1.1, SW2.1, U1.19 (GND), U1.20 (GND), U1.21 (GND), U1.22 (GND), U1.23 (GND), U1.24 (GND), U1.25 (GND), U1.26 (GND), U1.27 (GND), U1.9 (GND), U4.13 (GND), U4.5 (GND)
- net RS485_MODE: now also U1.10 (IO10)
- net RS485_RX: now also U1.6 (IO7)
- net RS485_TX: now also U1.5 (IO6)
- net STAT_LED: now also U1.3 (IO4)
- net USB_D+: now also U4.12 (USBDP)
- net USB_D-: now also U4.1 (USBDM)
- net at C6.1: now also R7.1, SW1.2, U1.2 (EN); no longer R7.2
- new net: C8.1, R9.1, U4.2 (*RESET)
- new net: SW2.2, U1.8 (IO9)
- new net FTDI_RX: U1.12 (TXD), U4.10 (RXD)
- new net FTDI_TX: U1.11 (RXD), U4.7 (TXD)
- new net IO8_PULLUP: R8.1, U1.16 (IO2), U1.7 (IO8)
- no-connect marks 10 -> 12
Other:
- moved on the sheet: D3, D4, R5, R6, U3

Commit message: Updated to revision 3.0
Parts:
- removed C8: 1uF, Capacitor_SMD:C_0805_2012Metric_Pad1.18x1.45mm_HandSolder, symbol Device:C
- removed SW1: RESET, Button_Switch_THT:SW_PUSH_6mm, symbol Switch:SW_Push
- removed SW2: BOOT, Button_Switch_THT:SW_PUSH_6mm, symbol Switch:SW_Push
- removed U4: FT234XD-R, USB-UART Bridge:FT234XD-R, symbol FTDI:FT234XD-R
- added D7: DBG_LED, LED_SMD:LED_0805_2012Metric_Pad1.15x1.40mm_HandSolder, symbol Device:LED
- added J2: Micro_SD_Card, Connector_Card:microSD_HC_Molex_47219-2001, symbol Connector:Micro_SD_Card
- added J3: Conn_01x02_Pin, Connector_PinHeader_2.54mm:PinHeader_1x02_P2.54mm_Vertical, symbol Connector:Conn_01x02_Pin
- added Q1, Q2: BC817, Package_TO_SOT_SMD:SOT-23, symbol Transistor_BJT:BC817
- added R10, R11, R12: 5.11K, Resistor_SMD:R_0805_2012Metric_Pad1.20x1.40mm_HandSolder, symbol Device:R_US
- added R13: 1M, Resistor_SMD:R_0805_2012Metric_Pad1.20x1.40mm_HandSolder, symbol Device:R_US
- added U4: FT231XQ, Package_DFN_QFN:QFN-20-1EP_4x4mm_P0.5mm_EP2.5x2.5mm, symbol Interface_USB:FT231XQ
- R9: value 5.11K -> 220
- renumbered TP3 to 3V3, TP2 to GND1, TP1 to VIN1
Connections:
- net +3.3V: now also J2.4 (VDD), R10.2, U4.10 (3V3OUT), U4.12 (VCC), U4.20 (VCCIO); no longer R9.2
- net FTDI_RX: now also U4.1 (RXD)
- net FTDI_TX: now also U4.17 (TXD)
- net GND: now also CONN1.3 (GND), R9.2, J2.6 (VSS), R13.2, U4.13 (GND), U4.21 (GND), U4.3 (GND); no longer CONN1.2 (GND)
- net RJ9_DA: now also CONN1.1 (DA); no longer CONN1.4 (DA)
- net RJ9_DB: now also CONN1.2 (DB); no longer CONN1.3 (DB)
- net USB_D+: now also U4.8 (USBDP)
- net USB_D-: now also U4.9 (USBDM)
- net EN_PU: now reaches C6.1, R7.1, U1.2 (EN)
- net EN_PU: now also J3.1 (Pin_1), Q1.3 (C)
- net at R9.1: now also D7.1 (K)
- net DBG_LED: now reaches U1.13 (IO18)
- net DBG_LED: now also D7.2 (A)
- net SD_SCL: now reaches U1.14 (IO19)
- net SD_SCL: now also J2.5 (CLK)
- net SD_CS: now reaches U1.15 (IO3)
- net SD_CS: now also J2.2 (DAT3/CD)
- net SD_MOSI: now reaches U1.17 (IO1)
- net SD_MOSI: now also J2.3 (CMD)
- net SD_MISO: now reaches U1.18 (IO0)
- net SD_MISO: now also J2.7 (DAT0)
- net IO9_BOOT: now reaches U1.8 (IO9)
- net IO9_BOOT: now also J3.2 (Pin_2), Q2.3 (C)
- net at C4.1, D5.2 (A): now also CONN1.4 (+12V); no longer CONN1.1 (+12V)
- new net: J2.9 (SHIELD), R13.1
- new net: Q2.2 (E), R11.1, U4.18 (~{DTR})
- new net: Q1.1 (B), R11.2
- new net: R10.1, U4.11 (~{RESET})
- new net: Q1.2 (E), R12.1, U4.19 (~{RTS})
- new net: Q2.1 (B), R12.2
- no-connect marks 12 -> 13
Other:
- note removed: "TODO Add comments on chips Check In/out capacitance on linear regulator Optimize w/ 5.11k? Check esp32 reflow spec"
- moved on the sheet: C6, D3, D4, R2, R5, R6, R7, R8
